File: ESP32_Base_PCB/ESP32-S3 Weather Station/ESP32-S3 Weather Station.kicad_pcb (KiCad board)
At the start: 2 copper layers, 31 parts, among them J1 USB_C_Receptacle_USB2.0_16P, Q1 Si2306, Q2 CSD19505, U1 AMS1117-3.3, U2 ESP32-S3-WROOM-2, U3 ADS1015IDGS, U5 IR2104, U6 AMS1117-5.0, U7 IR2104

Commit message: more changes
Parts:
- added BT1: 0-50V, TerminalBlock_MetzConnect:TerminalBlock_MetzConnect_Type703_RT10N02HGLU_1x02_P9.52mm_Horizontal, F.Cu at (58.5, 128.7)
- added C11: 47uF, Capacitor_SMD:C_0805_2012Metric_Pad1.18x1.45mm_HandSolder, F.Cu at (214.2, 102.4)
- added C12: 2.2uF, Capacitor_SMD:C_0805_2012Metric_Pad1.18x1.45mm_HandSolder, F.Cu at (214.2, 105.4)
- added C13: 2.2uF, Capacitor_SMD:C_0805_2012Metric_Pad1.18x1.45mm_HandSolder, F.Cu at (214.2, 108.4)
- added C14: 4.7uF, Capacitor_SMD:C_0805_2012Metric_Pad1.18x1.45mm_HandSolder, F.Cu at (214.2, 111.4)
- added C15: 100nF, Capacitor_SMD:C_0805_2012Metric_Pad1.18x1.45mm_HandSolder, F.Cu at (214.2, 114.5)
- added C16: 100nF, Capacitor_SMD:C_0805_2012Metric_Pad1.18x1.45mm_HandSolder, F.Cu at (214.2, 117.5)
- added C17: 10uF, Capacitor_SMD:C_0805_2012Metric_Pad1.18x1.45mm_HandSolder, F.Cu at (214.2, 120.5)
- added C18: 100nF, Capacitor_SMD:C_0805_2012Metric_Pad1.18x1.45mm_HandSolder, F.Cu at (219.0, 102.4)
- added C19: 100nF, Capacitor_SMD:C_0805_2012Metric_Pad1.18x1.45mm_HandSolder, F.Cu at (219.0, 105.4)
- added C20: 33nF, Capacitor_SMD:C_0805_2012Metric_Pad1.18x1.45mm_HandSolder, F.Cu at (219.0, 108.4)
- added C21: 100uF, Capacitor_SMD:C_0805_2012Metric_Pad1.18x1.45mm_HandSolder, F.Cu at (219.0, 111.4)
- added C22: 4.7uF, Capacitor_SMD:C_0805_2012Metric_Pad1.18x1.45mm_HandSolder, F.Cu at (219.0, 114.5)
- added C23: 4.7uF, Capacitor_SMD:C_0805_2012Metric_Pad1.18x1.45mm_HandSolder, F.Cu at (219.0, 117.5)
- added C24: 33nF, Capacitor_SMD:C_0805_2012Metric_Pad1.18x1.45mm_HandSolder, F.Cu at (219.0, 120.5)
- added C25: 100uF, Capacitor_SMD:C_0805_2012Metric_Pad1.18x1.45mm_HandSolder, F.Cu at (223.8, 102.4)
- added C26: 470uF, Capacitor_THT:CP_Radial_D16.0mm_P7.50mm, F.Cu at (83.8, 93.1)
- added C27: 100nF, Capacitor_SMD:C_0805_2012Metric_Pad1.18x1.45mm_HandSolder, F.Cu at (223.8, 108.4)
- added C28: 100uF, Capacitor_SMD:C_0805_2012Metric_Pad1.18x1.45mm_HandSolder, F.Cu at (146.7, 71.6)
- added C29: 470uF, Capacitor_THT:CP_Radial_D16.0mm_P7.50mm, F.Cu at (63.1, 93.1)
- added D10: SS310LW, Diode_SMD:D_SOD-123, F.Cu at (34.9, 74.8)
- added D11: LED, LED_SMD:LED_0805_2012Metric_Pad1.15x1.40mm_HandSolder, F.Cu at (40.1, 67.9)
- added D12: SS310LW, Diode_SMD:D_SOD-123, F.Cu at (34.9, 78.2)
- added D13: SS310LW, Diode_SMD:D_SOD-123, F.Cu at (34.9, 81.5)
- added D14: 1N4007, Diode_THT:D_DO-41_SOD81_P10.16mm_Horizontal, F.Cu at (213.7, 128.3)
- added D7: 1N4007, Diode_THT:D_DO-41_SOD81_P10.16mm_Horizontal, F.Cu at (213.7, 124.1)
- added D8: SS310LW, Diode_SMD:D_SOD-123, F.Cu at (34.9, 68.1)
- added D9: SS310LW, Diode_SMD:D_SOD-123, F.Cu at (34.9, 71.5)
- added F1: 35A, Fuse:Fuseholder_Keystone_3555-2, F.Cu at (211.0, 57.2)
- added F2: 35A, Fuse:Fuseholder_Keystone_3555-2, F.Cu at (211.0, 64.8)
- added L1: 60uH, Inductor_THT:L_Toroid_Vertical_L21.6mm_W11.4mm_P7.62mm_Pulse_KM-3, F.Cu at (259.0, 82.5)
- added L2: 100uH, B82442T1104K050:INDM5650X530N, F.Cu at (211.2, 71.8)
- added L3: 100uH, B82442T1104K050:INDM5650X530N, F.Cu at (211.2, 78.4)
- added Q3: CSD19505, Package_TO_SOT_THT:TO-220-3_Vertical, F.Cu at (96.9, 69.9)
- added Q4: CSD19505, Package_TO_SOT_THT:TO-220-3_Vertical, F.Cu at (108.1, 69.9)
- added R10: 10K, Resistor_SMD:R_0603_1608Metric_Pad0.98x0.95mm_HandSolder, F.Cu at (192.9, 138.8)
- added R11: 10K, Resistor_SMD:R_0603_1608Metric_Pad0.98x0.95mm_HandSolder, F.Cu at (192.9, 141.3)
- added R12: 10K, Resistor_SMD:R_0603_1608Metric_Pad0.98x0.95mm_HandSolder, F.Cu at (192.9, 143.8)
- added R13: 15K, Resistor_SMD:R_0603_1608Metric_Pad0.98x0.95mm_HandSolder, F.Cu at (197.2, 131.3)
- added R14: 100, Resistor_SMD:R_0603_1608Metric_Pad0.98x0.95mm_HandSolder, F.Cu at (197.2, 133.8)
- added R15: 100K, Resistor_SMD:R_0603_1608Metric_Pad0.98x0.95mm_HandSolder, F.Cu at (197.2, 136.3)
- added R16: 100, Resistor_SMD:R_0603_1608Metric_Pad0.98x0.95mm_HandSolder, F.Cu at (197.2, 138.8)
- added R17: 100K, Resistor_SMD:R_0603_1608Metric_Pad0.98x0.95mm_HandSolder, F.Cu at (197.2, 141.3)
- added R18: 10K, Resistor_SMD:R_0603_1608Metric_Pad0.98x0.95mm_HandSolder, F.Cu at (197.2, 143.8)
- added R19: 10K, Resistor_SMD:R_0603_1608Metric_Pad0.98x0.95mm_HandSolder, F.Cu at (201.6, 131.3)
- added R20: 100K, Resistor_SMD:R_0603_1608Metric_Pad0.98x0.95mm_HandSolder, F.Cu at (201.6, 133.8)
- added R21: 100K, Resistor_SMD:R_0603_1608Metric_Pad0.98x0.95mm_HandSolder, F.Cu at (201.6, 136.3)
- added R22: 15K, Resistor_SMD:R_0603_1608Metric_Pad0.98x0.95mm_HandSolder, F.Cu at (201.6, 138.8)
- added R23: 1K, Resistor_SMD:R_0603_1608Metric_Pad0.98x0.95mm_HandSolder, F.Cu at (201.6, 141.3)
- added R24: 15K, Resistor_SMD:R_0603_1608Metric_Pad0.98x0.95mm_HandSolder, F.Cu at (201.6, 143.8)
- added R25: 1K, Resistor_SMD:R_0603_1608Metric_Pad0.98x0.95mm_HandSolder, F.Cu at (205.9, 131.3)
- added R26: 15K, Resistor_SMD:R_0603_1608Metric_Pad0.98x0.95mm_HandSolder, F.Cu at (205.9, 133.8)
- added R27: 47K, Resistor_SMD:R_0603_1608Metric_Pad0.98x0.95mm_HandSolder, F.Cu at (205.9, 136.3)
- added R28: 1K, Resistor_SMD:R_0603_1608Metric_Pad0.98x0.95mm_HandSolder, F.Cu at (205.9, 138.8)
- added R29: 47K, Resistor_SMD:R_0603_1608Metric_Pad0.98x0.95mm_HandSolder, F.Cu at (205.9, 141.3)
- added R30: 10K, Resistor_SMD:R_0603_1608Metric_Pad0.98x0.95mm_HandSolder, F.Cu at (146.8, 67.9)
- added R7: 1K, Resistor_SMD:R_0603_1608Metric_Pad0.98x0.95mm_HandSolder, F.Cu at (192.9, 131.3)
- added R8: 3.3K, Resistor_SMD:R_0603_1608Metric_Pad0.98x0.95mm_HandSolder, F.Cu at (192.9, 133.8)
- added R9: 10K, Resistor_SMD:R_0603_1608Metric_Pad0.98x0.95mm_HandSolder, F.Cu at (192.9, 136.3)
- added SC1: 15V-80V, TerminalBlock_MetzConnect:TerminalBlock_MetzConnect_Type703_RT10N02HGLU_1x02_P9.52mm_Horizontal, F.Cu at (80.2, 128.6)
- added SW1: PTS810_SJM_250_SMTR_LFS, PTS815_SJG_250_SMTR_LFS:PTS815SJG250SMTRLFS, F.Cu at (230.8, 104.1)
- added SW2: PTS810_SJM_250_SMTR_LFS, PTS815_SJG_250_SMTR_LFS:PTS815SJG250SMTRLFS, F.Cu at (230.8, 110.4)
- added TH1: Thermistor_NTC, TerminalBlock:TerminalBlock_bornier-2_P5.08mm, F.Cu at (141.0, 69.9)
- moved J1 59.7 mm to (153.5, 140.0)
- moved Q2 57.8 mm to (86.0, 69.9)
- moved C10 53.0 mm to (116.3, 146.6)
- moved C2 53.0 mm to (111.5, 137.5)
- moved C3 53.0 mm to (111.5, 140.5)
- moved C5 53.0 mm to (111.5, 146.6)
- moved C7 53.0 mm to (116.3, 137.5)
- moved C8 53.0 mm to (116.3, 140.5)
- moved R2 53.0 mm to (106.9, 136.8)
- moved R3 53.0 mm to (106.9, 139.3)
- moved R5 53.0 mm to (106.9, 144.3)
- moved R6 53.0 mm to (106.9, 146.8)
- moved U1 53.0 mm to (99.8, 137.2)
- moved U5 53.0 mm to (147.5, 124.0)
- moved U6 53.0 mm to (99.8, 145.5)
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Connections:
- net AIN0 renamed A0
- C1 pad 1: VCC_5V -> Net-(D1-K)
- C2 pad 1: VCC_5V -> Net-(D1-K)
- C3 pad 1: VCC_5V -> Net-(D1-K)
- D1 pad 1: VCC_5V -> Net-(D1-K)
- Q1 pad 1: unconnected-(Q1-D-Pad1) -> Net-(PS1--VIN(GND))
- Q1 pad 2: unconnected-(Q1-G-Pad2) -> GPIO17
- Q1 pad 3: unconnected-(Q1-S-Pad3) -> GND
- Q2 pad 1: unconnected-(Q2-D-Pad1) -> Net-(Q2-D)
- Q2 pad 2: unconnected-(Q2-G-Pad2) -> Net-(PS1-+VOUT)
- Q2 pad 3: unconnected-(Q2-S-Pad3) -> Net-(D11-K)
- U1 pad 3: VCC_5V -> Net-(D1-K)
- U2 pad 10: unconnected-(U2-IO17-Pad10) -> GPIO17
- U2 pad 11: unconnected-(U2-IO18-Pad11) -> GPIO18
- U2 pad 8: unconnected-(U2-IO15-Pad8) -> GPIO15
- U2 pad 9: unconnected-(U2-IO16-Pad9) -> GPIO16
- U3 pad 5: AIN1 -> A1
- U3 pad 6: AIN2 -> A2
- U3 pad 7: AIN3 -> A3
- U6 pad 1: unconnected-(U6-GND-Pad1) -> GND
- U6 pad 2: unconnected-(U6-VO-Pad2) -> VCC_5V
- U6 pad 3: unconnected-(U6-VI-Pad3) -> +12V
- U7 pad 1: unconnected-(U7-VCC-Pad1) -> +12V
- U7 pad 2: unconnected-(U7-IN-Pad2) -> GPIO16
- U7 pad 3: unconnected-(U7-~{SD}-Pad3) -> GPIO15
- U7 pad 4: unconnected-(U7-COM-Pad4) -> GND
- U7 pad 5: unconnected-(U7-LO-Pad5) -> Net-(U7-LO)
- U7 pad 6: unconnected-(U7-VS-Pad6) -> Net-(Q3-S)
- U7 pad 7: unconnected-(U7-HO-Pad7) -> Net-(U7-HO)
- U7 pad 8: unconnected-(U7-VB-Pad8) -> Net-(U7-VB)
