File: ESP32_Base_PCB/Weather with charge/Weather with charge.kicad_pcb (KiCad board)
At the start: 2 copper layers, 120.8 x 60 mm, 40 parts, among them J1 USB_C_Receptacle_USB2.0_16P, J10 A3 of ADC, J11 External Power, J2 Rain Guage, J3 GPIO, J4 Wind Speed/DIR, J5 BME680, J6 Light Density, J7 Soil Mouisture, J8 I2C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

Commit message: now?
Parts:
- added C11: 10uF, Capacitor_SMD:C_0805_2012Metric_Pad1.18x1.45mm_HandSolder, F.Cu at (70.4, 56.3)
- added C12: 10uF, Capacitor_SMD:C_0805_2012Metric_Pad1.18x1.45mm_HandSolder, F.Cu at (70.4, 59.3)
- added C13: 1uF, Capacitor_SMD:C_0805_2012Metric_Pad1.18x1.45mm_HandSolder, F.Cu at (70.4, 62.3)
- added C14: 10uF, Capacitor_SMD:C_0805_2012Metric_Pad1.18x1.45mm_HandSolder, F.Cu at (70.4, 65.3)
- added D10: 10BQ040, Diode_SMD:D_SMA, F.Cu at (72.1, 76.2)
- added D11: 10BQ040, Diode_SMD:D_SMA, F.Cu at (72.1, 80.7)
- added D7: 1N4148, Diode_THT:D_DO-35_SOD27_P7.62mm_Horizontal, F.Cu at (69.6, 68.6)
- added D8: 1N4148, Diode_THT:D_DO-35_SOD27_P7.62mm_Horizontal, F.Cu at (69.6, 72.1)
- added D9: BZX84C6V2L, Package_TO_SOT_SMD:SOT-23, F.Cu at (75.3, 62.9)
- added J12: Battery, TerminalBlock_Phoenix:TerminalBlock_Phoenix_MKDS-1,5-2-5.08_1x02_P5.08mm_Horizontal, F.Cu at (59.4, 72.9)
- added J9: Solar Panel Input, TerminalBlock_Phoenix:TerminalBlock_Phoenix_MKDS-1,5-2-5.08_1x02_P5.08mm_Horizontal, F.Cu at (59.4, 61.0)
- added R10: 499K, Resistor_SMD:R_0603_1608Metric_Pad0.98x0.95mm_HandSolder, F.Cu at (53.6, 56.0)
- added R11: 100K, Resistor_SMD:R_0603_1608Metric_Pad0.98x0.95mm_HandSolder, F.Cu at (53.6, 58.5)
- added R12: 1M, Resistor_SMD:R_0603_1608Metric_Pad0.98x0.95mm_HandSolder, F.Cu at (53.6, 61.0)
- added R13: 174K, Resistor_SMD:R_0603_1608Metric_Pad0.98x0.95mm_HandSolder, F.Cu at (53.6, 63.5)
- added R14: 910, Resistor_SMD:R_0603_1608Metric_Pad0.98x0.95mm_HandSolder, F.Cu at (53.6, 66.1)
- added R15: 309K, Resistor_SMD:R_0603_1608Metric_Pad0.98x0.95mm_HandSolder, F.Cu at (53.6, 68.6)
- added R16: 100K, Resistor_SMD:R_0603_1608Metric_Pad0.98x0.95mm_HandSolder, F.Cu at (53.6, 71.1)
- added R17: 0.1, Resistor_SMD:R_0603_1608Metric_Pad0.98x0.95mm_HandSolder, F.Cu at (53.6, 73.6)
- added R18: 10K, Resistor_SMD:R_0603_1608Metric_Pad0.98x0.95mm_HandSolder, F.Cu at (53.6, 76.1)
- added R19: 7.15K, Resistor_SMD:R_0603_1608Metric_Pad0.98x0.95mm_HandSolder, F.Cu at (53.6, 78.6)
- added TH1: Thermistor_US, Resistor_SMD:R_0603_1608Metric, F.Cu at (78.1, 75.2)
- added U4: LT3652IMSE, Package_SO:MSOP-12-1EP_3x4mm_P0.65mm_EP1.65x2.85mm, F.Cu at (76.5, 57.7)
Connections:
- U2 pad 19: unconnected-(U2-IO11-Pad19) -> CHARGING
- U2 pad 20: unconnected-(U2-IO12-Pad20) -> CHARGE FAULT
